File: MotorBoard_v7/MotorBoard.kicad_pcb (KiCad board)
At the start: 2 copper layers, 98.9 x 86.4 mm, 61 parts, among them J1 5Vsel, J10 XDS_VCC, J13 Bump_Left, J14 Bump_Center, J15 Bump_Right, J2 1725656, J2_J4 LaunchPad, J3 CAN endpoint, J3_J1 LaunchPad, J4 1725656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

Commit message: added lab 6 update starter files
Parts:
- added C10: 4.7uF, ECE445L:C_0805_2012Metric, F.Cu at (139.8, 48.8)
- added C11: 4.7uF, ECE445L:C_0805_2012Metric, F.Cu at (139.8, 44.2)
- added TP12: +3.3V_ESP, ECE445L:Testpoint_1x1, F.Cu at (131.4, 40.4)
- added U4: LM2937ESX-3.3_NOPB, ECE445L:SOT230P700X180-4N, F.Cu at (133.2, 46.5)
- R1: value 1.6k -> 3.3k
- R2: value 750 -> 1.5k
- U3: footprint RSLK2:SSD1306 -> ECE445L:SSD1306
- moved R3 15.9 mm to (127.8, 40.8), turned to 90 degrees
- moved R5 10.3 mm to (112.0, 113.3)
- moved U5 4.19 mm to (123.1, 42.9)
- moved U3 1.27 mm to (104.4, 114.4)
Connections:
- R3 pad 1: +3V3 -> +3.3V_ESP
- U3 pad 1: GND -> +3V3
- U3 pad 2: +3V3 -> GND
- U3 pad 5: +3V3 -> GND
- U3 pad 6: GND -> +3V3
- U5 pad 1: PA17 -> PB17
- U5 pad 2: +3V3 -> +3.3V_ESP
- U5 pad 5: PA18 -> PB18
- U5 pad 8: +3V3 -> +3.3V_ESP
Routing:
- net PA17: track 102.3 -> 0.00 mm, vias 4 -> 0
- net PA18: track 74.2 -> 0.00 mm, vias 3 -> 0
- net PB17: track 0.00 -> 70.9 mm, vias 0 -> 2
- net PB18: track 0.00 -> 68.9 mm, vias 0 -> 3
- net +3V3: track 299.9 -> 233.7 mm
- net +5V: track 146.8 -> 201.8 mm, vias 3 -> 5
- net +3.3V_ESP: track 0.00 -> 25.8 mm
- net GND: track 83.4 -> 102.1 mm, vias 12 -> 13
- net PB3: track 33.1 -> 21.2 mm, vias 1 -> 2
- net PB2: track 39.0 -> 29.0 mm, vias 3 -> 2
- net Net-(U5-Ch_PD): track 6.75 -> 13.8 mm, vias 1 -> 2
- net Net-(J8-A): track 38.8 -> 43.3 mm
- net Net-(J8-B): track 50.3 -> 54.5 mm
- net PA25: track 102.7 -> 98.7 mm
- net PB19: track 78.3 -> 75.9 mm, vias 4 -> 3
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Other:
- board text added: "33uH"
- board text added: "ECE445M Motor Board Version 7.1"
- board text added: "PB17"
- board text added: "PB18"
- board text added: "PB6"
- board text added: "SSD1306"
- board text removed: "ECE445M Motor Board Version 7"
- board text removed: "PA17"
- board text removed: "PA18"
